File: fx3.kicad_sch (KiCad schematic)
At the start: 67 parts, among them J3 JTAG, J4 UART, SW1 RESET, U1 CYUSB3014-BZXI, U3 24LC1025-I/SN, U4 24LC1025-I/SN, Y1 19.2MHz

Commit message: PIO sheet: GPIO37 drives SBEN through 1k
Pin 5 is GND on a stock console, so a GPIO37 driven high sinks 3.3 mA
instead of shorting it. check_netlist checks the hop like /RESET and /CS2.
Parts:
- removed R8: 10k, Resistor_SMD:R_0402_1005Metric, symbol Device:R
- added R24: 100, Resistor_SMD:R_0402_1005Metric, symbol Device:R
- R11: now not fitted
- R12, R9: now fitted
- R15: value 1k -> 10k; LCSC C11702 -> C25744; now not fitted
- R16: value 10k -> 1k; LCSC C25744 -> C11702
- R17: value 2k -> 10k; LCSC C4109 -> C25744
- R19: value 6.04k 1% -> 2k; LCSC C97819 -> C4109
- R20: value 200 1% -> 6.04k 1%; LCSC C25087 -> C97819
- R21: value 470 -> 200 1%; LCSC C25117 -> C25087
- R22: value 100 -> 470; LCSC C25076 -> C25117
Connections:
- net +3V3: now also R10.2, R12.2, R14.2, R16.2, R19.2; no longer R11.2, R13.2, R15.2, R17.2, R9.2
- net FX3_CVDDQ: now also R17.2; no longer R16.2
- net FX3_FSLC: now also R9.1
- net FX3_PMODE0: now also R11.1; no longer R9.1
- net FX3_PMODE0_UP: now also R16.1; no longer R15.1
- net FX3_PMODE1: now also R13.1; no longer R11.1
- net FX3_PMODE2: now also R15.1; no longer R13.1
- net FX3_RESETn: now also R17.1; no longer R16.1
- net FX3_RUSB2: now also R20.1; no longer R19.1
- net FX3_RUSB3: now also R21.1; no longer R20.1
- net GND: now also R11.2, R13.2, R15.2, R21.2, R9.2; no longer R10.2, R12.2, R14.2, R19.2
- net I2C_SCL: now also R18.1; no longer R17.1
- net I2C_SDA: now also R19.1; no longer R18.1
- net LED_B: now also R24.2; no longer R23.2
- net LED_B_K: now also R24.1; no longer R23.1
- net LED_G: now also R23.2; no longer R22.2
- net LED_G_K: now also R23.1; no longer R22.1
- net LED_R: now also R22.2; no longer R21.2
- net LED_R_K: now also R22.1; no longer R21.1
- net PIO_SBEN renamed PIO_SBEN_DRV
