File: power.kicad_sch (KiCad schematic)
At the start: 11 parts, among them U5 TLV62569DBVR

Commit message: PIO sheet: GPIO37 drives SBEN through 1k
Pin 5 is GND on a stock console, so a GPIO37 driven high sinks 3.3 mA
instead of shorting it. check_netlist checks the hop like /RESET and /CS2.
Parts:
- removed R25: 100k, Resistor_SMD:R_0402_1005Metric, symbol Device:R
- added R28: 1k, Resistor_SMD:R_0402_1005Metric, symbol Device:R
- R27: value 1k -> 100k; LCSC C11702 -> C25741
Connections:
- net +1V2: now also R26.1
- net FB_1V2: now also R26.2, R27.1; no longer R26.1
- net GND: now also R28.2; no longer R26.2
- net PWR_LED_K: now also R28.1; no longer R27.1
