File: usb.kicad_sch (KiCad schematic)
At the start: 8 parts, among them J2 ZX360D-B-10P

Commit message: PIO sheet: GPIO37 drives SBEN through 1k
Pin 5 is GND on a stock console, so a GPIO37 driven high sinks 3.3 mA
instead of shorting it. check_netlist checks the hop like /RESET and /CS2.
Parts:
- removed R24: 100k, Resistor_SMD:R_0402_1005Metric, symbol Device:R
- added R25: 100k, Resistor_SMD:R_0402_1005Metric, symbol Device:R
Connections:
- net GND: now also R25.2
- net USB3_SHIELD: now also R25.1
